File: XDS-QuadAES-Studiohub.sch (KiCad schematic (older format))
At the start: 4 parts, among them J1 WeurthRJ45-8p8c-2x2-615032243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, J2 DB9_Male_MountingHoles

Commit message: minor changes
Parts:
- J1: footprint 615032243321 -> kicad:615032243321
- J2: value DB9_Male_MountingHoles -> DB9_Female; footprint Connector_Dsub:DSUB-9_Female_Horizontal_P2.77x2.84mm_EdgePinOffset4.94mm_Housed_MountingHolesOffset7.48mm -> Connector_Dsub:DSUB-9_Female_Horizontal_P2.77x2.84mm_EdgePinOffset7.70mm_Housed_MountingHolesOffset9.12mm
Changed lines of the file:
@@
 P 5400 3050
 F 0 "J2" H 5580 3052 50  0000 L CNN
-F 1 "DB9_Male_MountingHoles" H 5580 2961 50  0000 L CNN
-F 2 "Connector_Dsub:DSUB-9_Female_Horizontal_P2.77x2.84mm_EdgePinOffset4.94mm_Housed_MountingHolesOffset7.48mm" H 5400 3050 50  0001 C CNN
+F 1 "DB9_Female" H 5580 2961 50  0000 L CNN
+F 2 "Connector_Dsub:DSUB-9_Female_Horizontal_P2.77x2.84mm_EdgePinOffset7.70mm_Housed_MountingHolesOffset9.12mm" H 5400 3050 50  0001 C CNN
 F 3 " ~" H 5400 3050 50  0001 C CNN
 	1    5400 3050
@@
 F 0 "J1" H 2427 4037 50  0000 L CNN
 F 1 "WeurthRJ45-8p8c-2x2-615032243321" H 2427 3946 50  0000 L CNN
-F 2 "615032243321" H 1950 4000 50  0001 L BNN
+F 2 "kicad:615032243321" H 1950 4000 50  0001 L BNN
 F 3 "" H 1950 4000 50  0001 L BNN
 F 4 "615032243321" H 1950 4000 50  0001 L BNN "VALUE"
@@
 F 0 "J1" H 2427 2737 50  0000 L CNN
 F 1 "WeurthRJ45-8p8c-2x2-615032243321" H 2427 2646 50  0000 L CNN
-F 2 "615032243321" H 1950 2700 50  0001 L BNN
+F 2 "kicad:615032243321" H 1950 2700 50  0001 L BNN
 F 3 "" H 1950 2700 50  0001 L BNN
 F 4 "615032243321" H 1950 2700 50  0001 L BNN "VALUE"
@@
 F 0 "J1" H 2427 5387 50  0000 L CNN
 F 1 "WeurthRJ45-8p8c-2x2-615032243321" H 2427 5296 50  0000 L CNN
-F 2 "615032243321" H 1950 5350 50  0001 L BNN
+F 2 "kicad:615032243321" H 1950 5350 50  0001 L BNN
 F 3 "" H 1950 5350 50  0001 L BNN
 F 4 "615032243321" H 1950 5350 50  0001 L BNN "VALUE"
@@
 F 0 "J1" H 2427 1437 50  0000 L CNN
 F 1 "WeurthRJ45-8p8c-2x2-615032243321" H 2427 1346 50  0000 L CNN
-F 2 "615032243321" H 1950 1400 50  0001 L BNN
+F 2 "kicad:615032243321" H 1950 1400 50  0001 L BNN
 F 3 "" H 1950 1400 50  0001 L BNN
 F 4 "615032243321" H 1950 1400 50  0001 L BNN "VALUE"
